Commit message: build changes

File: franka_driver/franka_description/robots/panda_schunk.urdf.xacro (robot description, xacro)
@@ -7,3 +7,6 @@
     <origin xyz="0 0 0" rpy="0 0 0.785" />
   </xacro:schunk_pg70>
+  <xacro:world_ref name="world" parent="panda_link0">
+    <origin xyz="-0.0 0.0 0.0" rpy=" 0.0 0.0 0.0" />
+  </xacro:world_ref>
 </robot>

Commit message: Add database_wires

File: franka_driver/franka_description/robots/panda_schunk.urdf.xacro (robot description, xacro)
@@ -7,6 +7,3 @@
     <origin xyz="0 0 0" rpy="0 0 0.785" />
   </xacro:schunk_pg70>
-  <xacro:world_ref name="world" parent="panda_link0">
-    <origin xyz="-0.0 0.0 0.0" rpy=" 0.0 0.0 0.0" />
-  </xacro:world_ref>
 </robot>
