Commit message: Correction of wrong moveit_config files

File: franka_driver/panda_schunk_moveit_config/config/panda_arm.srdf.xacro (robot description, xacro)
@@ -74,4 +74,5 @@
     <disable_collisions link1="panda_link5" link2="schunk_pg70_fingertip_right_link" reason="Default" />
     <disable_collisions link1="panda_link6" link2="panda_link7" reason="Adjacent" />
+    <disable_collisions link1="panda_link6" link2="panda_link8" reason="Default" />
     <disable_collisions link1="panda_link6" link2="schunk_pg70_base_link" reason="Never" />
     <disable_collisions link1="panda_link6" link2="schunk_pg70_finger_left_link" reason="Never" />
@@ -98,3 +99,5 @@
     <disable_collisions link1="schunk_pg70_finger_right_link" link2="schunk_pg70_fingertip_right_link" reason="Adjacent" />
     <disable_collisions link1="schunk_pg70_fingertip_left_link" link2="schunk_pg70_fingertip_right_link" reason="Never" />
+    <disable_collisions link1="schunk_pg70_fingertip_right_link" link2="schunk_pg70_finger_left_link" reason="Default" />
+    <disable_collisions link1="schunk_pg70_fingertip_left_link" link2="schunk_pg70_finger_right_link" reason="Default" />
 </robot>

File: schunk_pg70/urdf/pg70.urdf.xacro (robot description, xacro)
@@ -113,4 +113,24 @@
      </collision>
     </link>
+<!-- OBJECT POSITION-->
+    <joint name="${name}_object_joint" type="fixed" >
+      <parent link="${name}_base_link" />
+      <child link="${name}_object_link" />
+      <origin xyz="0 0 0.18" rpy="0 0 0"/>
+   </joint>
+    <link name="${name}_object_link">
+      <visual>
+        <geometry>
+          <box size="0.0 0.00 0.0"/>
+        </geometry>
+	<material name="silver" />
+      </visual>
+      <collision>
+        <geometry>
+          <box size="0.00 0.00 0.0"/>
+        </geometry>
+	<material name="black"/>
+     </collision>
+    </link>
   </xacro:macro>
 </robot>

File: schunk_pg70/urdf/pg70_visualization.urdf.xacro (robot description, xacro)
@@ -7,3 +7,6 @@
     <origin xyz="0 0 0" rpy="0 0 0" />
   </xacro:schunk_pg70>
+  <xacro:schunk_pg70 name="object" parent="base_link">
+    <origin xyz="0 0 0.2" rpy="0 0 0" />
+  </xacro:schunk_pg70>
  </robot>
