Commit message: Add moveit config of schunk gripepr

File: schunk_pg70/urdf/pg70.urdf.xacro (robot description, xacro)
@@ -21,5 +21,5 @@
           <mesh filename="package://schunk_pg70/meshes/pg70.dae" />
         </geometry>
-	<material name="blue"/>
+	      <material name="blue"/>
       </collision>
     </link>

Commit message: final v

File: schunk_pg70/urdf/pg70.urdf.xacro (robot description, xacro)
@@ -117,5 +117,5 @@
       <parent link="${name}_base_link" />
       <child link="${name}_object_link" />
-      <origin xyz="0 0 0.18" rpy="0 0 0"/>
+      <origin xyz="0 0 0.21" rpy="0 0 0"/>
    </joint>
     <link name="${name}_object_link">

Commit message: Cyclic test file

File: schunk_pg70/urdf/pg70.urdf.xacro (robot description, xacro)
@@ -117,5 +117,5 @@
       <parent link="${name}_base_link" />
       <child link="${name}_object_link" />
-      <origin xyz="0 0 0.21" rpy="0 0 0"/>
+      <origin xyz="0 0 0.215" rpy="0 0 0"/>
    </joint>
     <link name="${name}_object_link">
